File: FastDataAcqSch.brd (EAGLE design)
At the start: 160 x 100 mm, 94 parts, among them IC1 FT230XQ, J1 USB_MICROAB_SMT, X1 SMA-SMDRA, X2 87832-14, Y1 SI530-500

Commit message: Update 9/2/13
Added more ICs
Parts:
- added C62, C64, C66, C68: .1uF, Schuyler:0204REVERSE
- added C63, C65: 10nF, rcl:C0201
- added C67: 100pF, rcl:C0603
- added C69: 4.7uF, Schuyler:0306REVERSE
- added R19, R20, R24, R25: 10k, rcl:R0201
- added R21: 1k, rcl:0204V
- added R22: 83, rcl:0204V
- added R23: 130, rcl:0204V
- added U$6: TMP421, Schuyler:SOT23-8
- added U$7: DAC101C081, Schuyler:SOT23-6
- added Y2: DNP, Schuyler:SI500S
- added Y3: 100MHz, Schuyler:UMAX8
Connections:
- new net FPGA_CLK1: U$2.P$55, Y3.P$1
- new net FPGA_CLK2: U$2.P$51, Y2.P$3
- new net FPGA_SCL: R19.1, R24.1, U$2.P$43, U$6.P$7, U$7.P$5
- new net FPGA_SDA: R20.1, R25.1, U$6.P$6, U$7.P$4
- new net FPGA_SDL: U$2.P$44
- new net N$10: R21.1
- new net N$9: R21.2, R22.2, R23.1
- new net VCC: R23.2
- net 3V3: now also C62.P$1, C63.1, C64.P$1, C65.1, C66.P$1, C68.P$1, C69.P$1, R19.2, R20.2, R24.2, R25.2, U$6.P$8, U$7.P$2, Y2.P$1, Y2.P$4, Y3.P$2, Y3.P$3, Y3.P$6
- net ADC_TDIODE+: now also C67.1, U$6.P$1
- net ADC_TDIODE-: now also C67.2, U$6.P$2
- net AGND: now also R22.1
- net DGND: now also C62.P$2, C63.2, C64.P$2, C65.2, C66.P$2, C68.P$2, C69.P$2, U$6.P$3, U$6.P$4, U$6.P$5, U$7.P$3, U$7.P$6, Y2.P$2, Y3.P$4, Y3.P$5

Commit message: Nearly finalized schematic
Parts:
- removed R21: 1k, rcl:0204V
- removed R22: 83, rcl:0204V
- removed R23: 130, rcl:0204V
- removed R9: NA, rcl:R0603
- added C70, C71, C72, C73, C74, C75, C76, C77, C78, C97, C98, C99: 10uF, rcl:C0603
- added C79, C80, C81, C82, C83, C84, C85, C93: 33uF, SparkFun-Passives:0805
- added C86, C87, C88, C89, C90, C91: 10pF, rcl:C0201
- added C92: 10nF, rcl:C0201
- added C94, C95, C96: 22uF 150mOhm ESR, rcl:C0805
- added IC2: LT1963AEQ, linear-technology:Q5-DD
- added JP1: (no value), SparkFun-Passives:1X02
- added L10, L11: 2.2uH, Schuyler:5.18X5.49_VISHAY
- added L6, L7, L8, L9: 2.2uH, Schuyler:3.0X3.6_VISHAY
- added R26, R27, R28, R29, R30, R31, R32, R33, R34, R35, R36, R37, R38, R41, R42, R43, R44, R45, R47, R48, R49: (no value), rcl:R0201
- added R39: 4.7k, rcl:R0201
- added R40: 0, rcl:R0603
- added R46, R50: (no value), rcl:R0603
- added R51: 10k, rcl:R0201
- added TP1, TP2, TP3, TP4, TP5, TP6, TP7, TP8, TP9: TPPAD1-13, testpad:P1-13
- added U$10: LT1963AEST-3.3, Schuyler:SOT223
- added U$8: LTC3374QFN, Schuyler:38-QFN_(5X7)
- added U$9: LT1963AEST-2.5, Schuyler:SOT223
- R1: device rcl:R0402 -> rcl:R0201
- moved R1 565.5 mm to (-160.5, -676.1)
Connections:
- removed net FGPA_PROGRAMB: U$2.P$37
- removed net N$10: R21.1
- removed net N$9: R21.2, R22.2, R23.1
- new net 2V3_1V9PRE: C82.1, C89.1, C97.1, IC2.1, IC2.2, L10.P$2, R32.2, TP3.TP
- new net 2V8_2V5PRE: C80.1, C91.1, C98.1, L9.P$2, R36.2, R48.2, TP1.TP, U$9.1
- new net 3V3A: C96.1, L4.P$2, TP9.TP, U$10.3
- new net 3V6_PRE3V3: C84.1, C87.1, C99.1, L6.P$2, R28.2, TP5.TP, U$10.1
- new net ADC_PWR_EN: R41.2, U$2.P$48, U$8.P$19
- new net ANALOG_PWR_EN: R47.2, U$2.P$47, U$8.P$32
- new net FPGA_PROGRAMB: R39.1, R40.2, U$2.P$37
- new net N$11: R40.1, U$5.P$7
- new net N$12: R42.1, R43.2, U$8.P$38
- new net N$13: R44.1, R45.2, U$8.P$13
- new net N$14: IC2.5, R46.1, R50.2
- new net N$16: R48.1, R49.2, U$8.P$14
- new net PGOOD: U$8.P$15
- new net S1FB: C86.2, R26.1, R27.2, U$8.P$1
- new net S1SW: L11.P$1, U$8.P$3, U$8.P$4
- new net S3FB: C87.2, R28.1, R29.2, U$8.P$7
- new net S3SW: L6.P$1, U$8.P$9
- new net S4FB: C88.2, R30.1, R31.2, U$8.P$12
- new net S4SW: L7.P$1, U$8.P$10
- new net S5FB: C89.2, R32.1, R33.2, U$8.P$20
- new net S5SW: L10.P$1, U$8.P$22, U$8.P$23
- new net S7FB: C90.2, R34.1, R35.2, U$8.P$26
- new net S7SW: L8.P$1, U$8.P$28
- new net S8FB: C91.2, R36.1, R37.2, U$8.P$31
- new net S8SW: L9.P$1, U$8.P$29
- new net S_TEMP: U$8.P$36
- new net VIN: C70.1, C71.1, C72.1, C73.1, C74.1, C75.1, C76.1, C77.1, C78.1, C79.1, U$8.P$11, U$8.P$17, U$8.P$2, U$8.P$21, U$8.P$24, U$8.P$25, U$8.P$27, U$8.P$30, U$8.P$33, U$8.P$35, U$8.P$5, U$8.P$6, U$8.P$8
- net 1V2: now also C81.1, C90.1, L8.P$2, R34.2, R42.2, TP2.TP
- net 1V8: now also C83.1, C88.1, L7.P$2, R30.2, TP4.TP
- net 1V9: now also C94.1, IC2.4, R46.2, TP7.TP
- net 1V9A: now also R51.2; no longer R9.2
- net 2V5: now also C95.1, TP8.TP, U$9.3
- net 3V3: now also C85.1, C86.1, C92.1, C93.1, L11.P$2, R26.2, R39.2, R44.2, TP6.TP; no longer L4.P$2
- net ADC_CALDLY/DES/!SCS: now also R51.1; no longer R9.1
- net AGND: now also R1.1; no longer R1.2, R22.1
- net DGND: now also C70.2, C71.2, C72.2, C73.2, C74.2, C75.2, C76.2, C77.2, C78.2, C79.2, C80.2, C81.2, C82.2, C83.2, C84.2, C85.2, C92.2, C93.2, C94.2, C95.2, C96.2, C97.2, C98.2, C99.2, IC2.3, IC2.6, R27.1, R29.1, R31.1, R33.1, R35.1, R37.1, R38.1, R41.1, R43.1, R45.1, R47.1, R49.1, R50.1, U$10.2, U$10.4, U$8.P$16, U$8.P$18, U$8.P$37, U$8.P$39, U$9.2, U$9.4
- net FPGA_CLK2: now also U$2.P$56; no longer U$2.P$51
- net N$2: now also R1.2; no longer R1.1
- net N$6: now also JP1.1, R38.2, U$8.P$34; no longer U$2.P$35
- net VCC: now also JP1.2; no longer R23.2

Commit message: Only 9 parts left to source
Parts:
- removed R18: 300, rcl:R0201
- removed R24, R25, R51: 10k, rcl:R0201
- added R21, R22, R9: 10k, rcl:R0201
- added R23: 330, rcl:R0201
- R17: value 300 -> 330
- R26: value (none) -> 845k
- R27: value (none) -> 270k
- R28, R32, R36: value (none) -> 523K
- R29: value (none) -> 150K
- R3, R4: device rcl:R0201 -> rcl:R0402
- R30: value (none) -> 806K
- R31: value (none) -> 649K
- R33: value (none) -> 280K
- R34, R37: value (none) -> 210K
- R35: value (none) -> 422K
- R46: value (none) -> 1.15k 1%
- R50: value (none) -> 2k 1%
- moved R4 561.5 mm to (-160.1, -709.3)
- moved R14 487.2 mm to (-160.5, -685.6)
- moved R17 447.6 mm to (-160.5, -718.8)
- moved R20 390.3 mm to (-160.5, -695.1)
- moved R19 390.3 mm to (-160.5, -690.3)
Connections:
- net 1V9A: now also R22.2, R9.1; no longer R14.1, R51.2
- net 3V3: now also R21.2; no longer R20.2, R24.2, R25.2
- net ADC_CAL: now also R9.2; no longer R14.2
- net ADC_CALDLY/DES/!SCS: now also R22.1; no longer R51.1
- net FPGA_RXD: now also R23.2; no longer R17.2
- net FPGA_SCL: no longer R19.1, R24.1
- net FPGA_SDA: now also R19.1, R21.1; no longer R20.1, R25.1
- net FPGA_TXD: now also R17.2; no longer R18.2
- net FTDI_RXD: now also R17.1; no longer R18.1
- net FTDI_TXD: now also R23.1; no longer R17.1

Commit message: Schematic Finalized
Parts:
- added C100, C101: .1uF, Schuyler:0204REVERSE
- added C102: 4.7uF, Schuyler:0306REVERSE
- added IC3: ADCMP553BRMZ, Schuyler:SOP65P490X110-8N
- added R18, R24: 150K, rcl:R0201
- added R25: 210K, rcl:R0201
- added R51: 16k, rcl:R0603
- added R52, R53, R54: 50, rcl:R0201
- added R55: 100, rcl:R0603
- added X3: SMA-142-0701-801/806, con-coax:J502-ND-142-0701-801/806
- C1, C12, C13, C15, C17, C2, C22, C4, C6, C7: value .1uF -> 10uF; device Schuyler:0204REVERSE -> rcl:C0603
- C10, C11, C19, C28, C29, C3: value .1uF -> 33uF; device Schuyler:0204REVERSE -> SparkFun-Passives:0805
- C14, C26, C8, C9: value .1uF -> 10pF; device Schuyler:0204REVERSE -> rcl:C0201
- C16, C18, C5: value .1uF -> NA; device Schuyler:0204REVERSE -> rcl:C0603
- C20, C21: value 33uF -> 10uF; device SparkFun-Passives:0805 -> rcl:C0603
- C23: value 1uF -> 22uF 150mOhm ESR; device Schuyler:0204REVERSE -> rcl:C0805
- C24: value 4.7nF -> 22uF 150mOhm ESR; device rcl:C0201 -> rcl:C0805
- C25: value 4.7nF -> 10pF
- C27: value 33uF -> 10pF; device SparkFun-Passives:0805 -> rcl:C0201
- C30: value 0.47uF -> 33uF; device Schuyler:0306REVERSE -> SparkFun-Passives:0805
- C31: value 4.7uF -> 22uF 150mOhm ESR; device Schuyler:0306REVERSE -> rcl:C0805
- C36, C37, C42, C45, C56: value 4.7uF -> 0.47uF
- C38, C39: value 4.7uF -> 33uF; device Schuyler:0306REVERSE -> SparkFun-Passives:0805
- C43, C44, C46, C47, C49, C53: value 0.47uF -> .1uF; device Schuyler:0306REVERSE -> Schuyler:0204REVERSE
- C48, C69: value 4.7uF -> .1uF; device Schuyler:0306REVERSE -> Schuyler:0204REVERSE
- C50, C52: value 0.47uF -> 4.7uF
- C55: value 1uF -> 0.47uF; device Schuyler:0204REVERSE -> Schuyler:0306REVERSE
- C57, C68: value .1uF -> 4.7uF; device Schuyler:0204REVERSE -> Schuyler:0306REVERSE
- C59: value 47pF -> .1uF; device rcl:C0201 -> Schuyler:0204REVERSE
- C60: value 47pF -> 4.7uF; device rcl:C0201 -> Schuyler:0306REVERSE
- C61: value 10nF -> 0.47uF; device rcl:C0201 -> Schuyler:0306REVERSE
- C62: value .1uF -> 0.47uF; device Schuyler:0204REVERSE -> Schuyler:0306REVERSE
- C63: value 10nF -> .1uF; device rcl:C0201 -> Schuyler:0204REVERSE
- C65: value 10nF -> 4.7uF; device rcl:C0201 -> Schuyler:0306REVERSE
- C67: value 100pF -> .1uF; device rcl:C0603 -> Schuyler:0204REVERSE
- C70, C72, C73, C75, C78, C97: value 10uF -> .1uF; device rcl:C0603 -> Schuyler:0204REVERSE
- C71, C74: value 10uF -> 4.7uF; device rcl:C0603 -> Schuyler:0306REVERSE
- C76: value 10uF -> 0.47uF; device rcl:C0603 -> Schuyler:0306REVERSE
- C77: value 10uF -> 100pF
- C79, C82, C83, C85, C93: value 33uF -> .1uF; device SparkFun-Passives:0805 -> Schuyler:0204REVERSE
- C80, C81: value 33uF -> 4.7nF; device SparkFun-Passives:0805 -> rcl:C0201
- C86: value 10pF -> 1uF; device rcl:C0201 -> Schuyler:0204REVERSE
- C87: value 10pF -> 33uF; device rcl:C0201 -> SparkFun-Passives:0805
- C88: value 10pF -> 4.7uF; device rcl:C0201 -> Schuyler:0306REVERSE
- C89, C91: value 10pF -> .1uF; device rcl:C0201 -> Schuyler:0204REVERSE
- C90: value 10pF -> 10nF
- C94, C95: value 22uF 150mOhm ESR -> 10nF; device rcl:C0805 -> rcl:C0201
- C96: value 22uF 150mOhm ESR -> 47pF; device rcl:C0805 -> rcl:C0201
- C98: value 10uF -> 47pF; device rcl:C0603 -> rcl:C0201
- C99: value 10uF -> 1uF; device rcl:C0603 -> Schuyler:0204REVERSE
- IC1: value FT230XQ -> LT1963AEQ; device ftdichip:QFN16 -> linear-technology:Q5-DD
- IC2: value LT1963AEQ -> FT230XQ; device linear-technology:Q5-DD -> ftdichip:QFN16
- L1, L2, L4: value 400@100MHz -> 2.2uH; device Schuyler:2220_FERRITE_BEAD -> Schuyler:3.0X3.6_VISHAY
- L10: value 2.2uH -> (none); device Schuyler:5.18X5.49_VISHAY -> Schuyler:2220_FERRITE_BEAD
- L11: value 2.2uH -> 600@100MHz; device Schuyler:5.18X5.49_VISHAY -> dp_devices:FB603
- L3: value (none) -> 2.2uH; device Schuyler:2220_FERRITE_BEAD -> Schuyler:5.18X5.49_VISHAY
- L5: value 600@100MHz -> 2.2uH; device dp_devices:FB603 -> Schuyler:3.0X3.6_VISHAY
- L6: device Schuyler:3.0X3.6_VISHAY -> Schuyler:5.18X5.49_VISHAY
- L7, L8, L9: value 2.2uH -> 400@100MHz; device Schuyler:3.0X3.6_VISHAY -> Schuyler:2220_FERRITE_BEAD
- R1: value 50 -> NA; device rcl:R0201 -> rcl:R0603
- R11: value NA -> 649K; device rcl:R0603 -> rcl:R0201
- R12: value NA -> 150K; device rcl:R0603 -> rcl:R0201
- R13: value 10k -> NA; device rcl:R0201 -> rcl:R0603
- R14, R19: value 10k -> 523K
- R15, R16: value 27 -> 523K
- R17: value 330 -> 210K
- R2: value 330 -> NA; device rcl:R0201 -> rcl:R0603
- R20: value 10k -> 280K
- R21: value 10k -> 270k
- R22: value 10k -> 210K
- R23: value 330 -> 806K
- R26: value 845k -> 806K
- R27: value 270k -> 845k
- R28: value 523K -> 649K
- R29: value 150K -> 422K
- R3: value 100 0.1% -> NA; device rcl:R0402 -> rcl:R0603
- R30: value 806K -> 270k
- R31: value 649K -> 1.15k 1%; device rcl:R0201 -> rcl:R0603
- R32: value 523K -> 2k 1%; device rcl:R0201 -> rcl:R0603
- R33: value 280K -> 50
- R34, R37: value 210K -> 10k
- R35: value 422K -> 10k
- R36: value 523K -> 10k
- R38: value (none) -> NA; device rcl:R0201 -> rcl:R0603
- R39: value 4.7k -> 100 0.1%; device rcl:R0201 -> rcl:R0402
- R4: value 100 0.1% -> 10k; device rcl:R0402 -> rcl:R0201
- R40: value 0 -> 100 0.1%; device rcl:R0603 -> rcl:R0402
- R41, R44, R45: value (none) -> 330
- R42: value (none) -> 4.7k
- R43: value (none) -> 0; device rcl:R0201 -> rcl:R0603
- R46: value 1.15k 1% -> 27; device rcl:R0603 -> rcl:R0201
- R47: value (none) -> 27
- R48: value (none) -> 10k; device rcl:R0201 -> rcl:R0603
- R49: value (none) -> 26.1k; device rcl:R0201 -> rcl:R0603
- R5: value 4.7k -> 10k
- R50: value 2k 1% -> 10k
- R6: value 3.3k 0.1% -> NA
- R7: value NA -> 3.3k 0.1%
- R8: value NA -> 10k; device rcl:R0603 -> rcl:R0201
- R9: value 10k -> 4.7k
- U$10: value LT1963AEST-3.3 -> XCFXXS04; device Schuyler:SOT223 -> Schuyler:TSSOP20_XILINX
- U$3: value LMH6555 -> LTC3374QFN; device Schuyler:16WQFN -> Schuyler:38-QFN_(5X7)
- U$4: value LMV321SC-70 -> LT1963AEST-2.5; device Schuyler:SC-70 -> Schuyler:SOT223
- U$5: value XCFXXS04 -> LT1963AEST-3.3; device Schuyler:TSSOP20_XILINX -> Schuyler:SOT223
- U$7: value DAC101C081 -> LMH6555; device Schuyler:SOT23-6 -> Schuyler:16WQFN
- U$8: value LTC3374QFN -> LMV321SC-70; device Schuyler:38-QFN_(5X7) -> Schuyler:SC-70
- U$9: value LT1963AEST-2.5 -> DAC101C081; device Schuyler:SOT223 -> Schuyler:SOT23-6
- X1: value SMA-SMDRA -> SMA-142-0701-801/806; device Schuyler:SMA-SMD2 -> con-coax:J502-ND-142-0701-801/806
- moved X1 874.5 mm to (-152.1, -805.2), turned to 0 degrees
- moved C5 758.0 mm to (-160.1, -756.8)
- moved U$10 723.3 mm to (141.2, 59.9), turned to 90 degrees
- moved U$5 723.3 mm to (-155.7, -599.6), turned to 0 degrees
- moved C24 717.4 mm to (-159.6, -642.2)
- moved C18 689.6 mm to (-160.1, -775.8)
- moved C16 685.6 mm to (-160.1, -771.1)
- moved U$4 673.4 mm to (-155.7, -587.3), turned to 0 degrees
- moved C21 617.5 mm to (-160.1, -666.6)
- moved C20 613.8 mm to (-160.1, -661.8)
- moved C25 581.4 mm to (-146.4, -505.2)
- moved R10 580.0 mm to (-160.1, -761.6)
- moved R13 571.9 mm to (-160.1, -766.3)
- moved C22 570.5 mm to (-160.1, -657.1)
- moved R11 567.2 mm to (-160.5, -752.1)
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Connections:
- removed net CLK_500_ENABLE: Y1.P$2
- removed net N$1: C22.P$1, C23.P$1, L3.P$1, Y1.P$6
- new net 2V5A: C85.P$1, C86.P$1, L10.P$1, Y1.P$2, Y1.P$6
- new net FPGA_TRIG+: IC3.6, R48.2, R53.2, U$2.P$51
- new net FPGA_TRIG-: IC3.5, R50.2, R52.2, U$2.P$50
- new net N$15: IC3.1, R48.1, R49.2
- new net N$18: R52.1, R53.1, R54.2
- new net N$20: IC3.2, R50.1, R51.2
- new net TRIGGER: IC3.3, X1.1
- new net TRIG_REF: IC3.4, U$9.P$1
- new net TRIG_RESET_HIGH: R51.1
- new net TRIG_RESET_LOW: R49.1
- net 1V2: now also C25.1, C28.1, C35.P$1, C40.P$1, C45.P$1, L4.P$2, R21.1, R25.2; no longer C30.P$1, C31.P$1, C33.P$1, C81.1, C90.1, L8.P$2, R34.2, R42.2
- net 1V8: now also C26.1, C29.1, L5.P$2, R26.2; no longer C83.1, C88.1, L7.P$2, R30.2
- net 1V9: now also C31.1, IC1.4, L7.P$1, L8.P$1, R31.2, R55.2; no longer C94.1, IC2.4, L1.P$1, L2.P$1, R46.2
- net 1V9A: now also C38.1, C43.P$1, C46.P$1, C48.P$1, C53.P$1, C58.P$1, C63.P$1, C66.P$1, C69.P$1, C72.P$1, C75.P$1, L7.P$2, R1.2, R4.1, R5.1, R6.2; no longer C1.P$1, C10.P$1, C2.P$1, C21.1, C3.P$1, C4.P$1, C5.P$1, C6.P$1, C7.P$1, C8.P$1, C9.P$1, L1.P$2, R11.2, R13.1, R22.2, R9.1
- net 1V9D: now also C39.1, C44.P$1, C47.P$1, C49.P$1, C54.P$1, C59.P$1, C64.P$1, C67.P$1, C70.P$1, C73.P$1, L8.P$2; no longer C11.P$1, C12.P$1, C13.P$1, C14.P$1, C15.P$1, C16.P$1, C17.P$1, C18.P$1, C19.P$1, C20.1, L2.P$2
- net 1V9F: now also C33.P$1, C36.P$1, C41.P$1, C50.P$1, C55.P$1, C56.P$1, C61.P$1, C62.P$1; no longer C42.P$1, C43.P$1, C44.P$1, C45.P$1, C46.P$1, C47.P$1, C52.P$1, C53.P$1
- net 2V3_1V9PRE: now also C14.1, C19.1, C22.1, IC1.1, IC1.2, L3.P$2, R19.2; no longer C82.1, C89.1, C97.1, IC2.1, IC2.2, L10.P$2, R32.2
- net 2V5: now also C23.1, L10.P$2, U$4.3; no longer C95.1, L3.P$2, U$9.3
- net 2V8_2V5PRE: now also C10.1, C20.1, C8.1, L1.P$2, R11.1, R15.2, U$4.1; no longer C80.1, C91.1, C98.1, L9.P$2, R36.2, R48.2, U$9.1
- net 3V3: now also C27.1, C30.1, C42.P$1, C52.P$1, C57.P$1, C60.P$1, C65.P$1, C71.P$1, C74.P$1, C76.P$1, C83.P$1, C87.1, C88.P$1, C89.P$1, C90.1, C91.P$1, C93.P$1, C94.1, C97.P$1, C99.P$1, IC3.7, L6.P$2, R23.2, R27.2, R35.2, R36.2, R37.2, R38.2, R41.2, R42.2, R9.2, U$10.P$18, U$10.P$19, U$10.P$20, U$9.P$2; no longer C35.P$1, C36.P$1, C38.P$1, C39.P$1, C40.P$1, C41.P$1, C48.P$1, C49.P$1, C50.P$1, C54.P$1, C55.P$1, C62.P$1, C63.1, C64.P$1, C65.1, C66.P$1, C69.P$1, C85.1, C86.1, C93.1, L11.P$2, R19.2, R2.2, R21.2, R26.2, R3.2, R44.2, R5.2, R7.2, U$5.P$18, U$5.P$19, U$5.P$20, U$7.P$2
- net 3V3A: now also C24.1, L9.P$2, U$5.3; no longer C96.1, L4.P$2, U$10.3
- net 3V3S: now also C78.P$1, C79.P$1, C82.P$1, C84.1, L9.P$1, U$7.P$11, U$7.P$12, U$7.P$9, U$8.P$5; no longer C26.P$1, C27.1, C28.P$1, C29.P$1, L4.P$1, U$3.P$11, U$3.P$12, U$3.P$9, U$4.P$5
- net 3V6_PRE3V3: now also C11.1, C21.1, C9.1, L2.P$2, R16.2, U$5.1; no longer C84.1, C87.1, C99.1, L6.P$2, R28.2, U$10.1
- net 5VUSB: now also C101.P$2, C102.P$1, IC2.10, L11.1; no longer C56.P$1, C57.P$2, IC1.10, L5.1
- net 5VUSB_CON: now also C95.1, L11.2; no longer C61.1, L5.2
- net ADC_CAL: now also R5.2; no longer R9.2
- net ADC_CALDLY/DES/!SCS: now also R8.1; no longer R22.1
- net ADC_CLK+: now also C80.2; no longer C24.2
- net ADC_CLK-: now also C81.2; no longer C25.2
- net ADC_DCLKRST: now also R3.2; no longer R12.2
- net ADC_FSR/ECE: now also R1.1, R2.2; no longer R10.2, R11.1
- net ADC_PD: now also R4.2; no longer R13.2
- net ADC_PWR_EN: now also R13.2, U$3.P$19; no longer R41.2, U$8.P$19
- net ADC_REXT: now also R7.2; no longer R6.2
- net ADC_TDIODE+: now also C77.1; no longer C67.1
- net ADC_TDIODE-: now also C77.2; no longer C67.2
- net ADC_VBG: now also R6.1; no longer R8.1
- net ADC_VCMO: now also U$8.P$1; no longer U$4.P$1
- net ADC_VCMO_BUFFER: now also U$7.P$10, U$8.P$3, U$8.P$4; no longer U$3.P$10, U$4.P$3, U$4.P$4
- net ADC_VINI+: now also U$7.P$8; no longer U$3.P$8
- net ADC_VINI-: now also U$7.P$13; no longer U$3.P$13
- net AGND: now also C38.2, C43.P$2, C46.P$2, C48.P$2, C53.P$2, C58.P$2, C63.P$2, C66.P$2, C69.P$2, C72.P$2, C75.P$2, C78.P$2, C79.P$2, C82.P$2, C84.2, C85.P$2, C86.P$2, R2.1, R3.1, R33.1, R7.1, U$7.P$1, U$7.P$14, U$7.P$15, U$7.P$17, U$7.P$2, U$7.P$3, U$7.P$4, U$7.P$6, U$7.P$7, U$8.P$2, X3.G@1, X3.G@2, X3.G@3, X3.G@4; no longer C1.P$2, C10.P$2, C2.P$2, C21.2, C22.P$2, C23.P$2, C26.P$2, C27.2, C28.P$2, C29.P$2, C3.P$2, C4.P$2, C5.P$2, C6.P$2, C7.P$2, C8.P$2, C9.P$2, R1.1, R10.1, R12.1, R6.1, U$3.P$1, U$3.P$14, U$3.P$15, U$3.P$17, U$3.P$2, U$3.P$3, U$3.P$4, U$3.P$6, U$3.P$7, U$4.P$2, X1.2@2, X1.2@3
- net ANALOG_PWR_EN: now also R10.2, U$3.P$32; no longer R47.2, U$8.P$32
- net CLK500+: now also C81.1; no longer C25.1
- net CLK500-: now also C80.1; no longer C24.1
- net DGND: now also C1.2, C10.2, C100.P$1, C101.P$1, C102.P$2, C11.2, C12.2, C13.2, C15.2, C16.2, C17.2, C18.2, C19.2, C2.2, C21.2, C22.2, C23.2, C24.2, C28.2, C29.2, C3.2, C30.2, C31.2, C39.2, C4.2, C5.2, C57.P$2, C59.P$2, C6.2, C60.P$2, C61.P$2, C65.P$2, C67.P$2, C7.2, C70.P$2, C71.P$2, C73.P$2, C74.P$2, C76.P$2, C83.P$2, C87.2, C88.P$2, C89.P$2, C90.2, C91.P$2, C93.P$2, C96.1, C97.P$2, C98.1, C99.P$2, IC1.6, IC3.8, R10.1, R12.2, R13.1, R14.1, R17.1, R18.1, R20.1, R22.1, R24.2, R28.1, R30.1, R32.1, R40.1, R54.1, R55.1, U$10.P$11, U$3.P$16, U$3.P$18, U$3.P$37, U$3.P$39, U$4.2, U$4.4, U$5.2, U$5.4, U$9.P$3, U$9.P$6; no longer C11.P$2, C12.P$2, C13.P$2, C14.P$2, C15.P$2, C16.P$2, C17.P$2, C18.P$2, C19.P$2, C30.P$2, C31.P$2, C38.P$2, C39.P$2, C43.P$2, C46.P$2, C48.P$2, C53.P$2, C57.P$1, C58.P$1, C59.1, C60.1, C61.2, C63.2, C65.2, C66.P$2, C69.P$2, C70.2, C71.2, C72.2, C73.2, C74.2, C75.2, C76.2, C77.2, C78.2, C79.2, C80.2, C81.2, C82.2, C83.2, C84.2, C85.2, C93.2, C96.2, C97.2, C98.2, C99.2, IC2.6, R27.1, R31.1, R33.1, R35.1, R37.1, R38.1, R4.1, R41.1, R43.1, R45.1, R47.1, R49.1, R50.1, U$10.2, U$10.4, U$5.P$11, U$7.P$3, U$7.P$6, U$8.P$16, U$8.P$18, U$8.P$37, U$8.P$39, U$9.2, U$9.4
- net FPGA_CCLK: now also R38.1, R39.1, R40.2, U$10.P$3; no longer R3.1, R4.2, R7.1, U$5.P$3
- net FPGA_DIN: now also U$10.P$1; no longer U$5.P$1
- net FPGA_DONE: now also R41.1, U$10.P$10; no longer R2.1, U$5.P$10
- net FPGA_INITB: now also R42.1, U$10.P$8; no longer R5.1, U$5.P$8
- net FPGA_PROGRAMB: now also R43.2, R9.1; no longer R39.1, R40.2
- net FPGA_RXD: now also R44.2; no longer R23.2
- net FPGA_SCL: now also R36.1, U$9.P$5; no longer U$7.P$5
- net FPGA_SDA: now also R35.1, R37.1, U$9.P$4; no longer R19.1, R21.1, U$7.P$4
- net FPGA_TCK: now also U$10.P$6; no longer U$5.P$6
- net FPGA_TDO: now also U$10.P$4; no longer U$5.P$4
- net FPGA_TMS: now also U$10.P$5; no longer U$5.P$5
- net FPGA_TXD: now also R45.2; no longer R17.2
- net FTDI_RXD: now also IC2.2, R45.1; no longer IC1.2, R17.1
- net FTDI_TXD: now also IC2.15, R44.1; no longer IC1.15, R23.1
- net GND: now also IC2.13; no longer IC1.13
- net N$11: now also R43.1, U$10.P$7; no longer R40.1, U$5.P$7
- net N$12: now also C18.1, R21.2, R22.2, U$3.P$38; no longer R42.1, R43.2, U$8.P$38
- net N$13: now also C16.1, R23.1, R24.1, U$3.P$13; no longer R44.1, R45.2, U$8.P$13
- net N$14: now also IC1.5, R31.1, R32.2; no longer IC2.5, R46.1, R50.2
- net N$16: now also C5.1, R11.2, R12.1, U$3.P$14; no longer R48.1, R49.2, U$8.P$14
- net N$2: now also R33.2, U$7.P$5; no longer R1.2, U$3.P$5
- net N$3: now also IC2.6, R46.2; no longer IC1.6, R15.2
- net N$4: now also C96.2, R46.1; no longer C59.2, R15.1
- net N$5: now also C98.2, R47.1; no longer C60.2, R16.1
- net N$6: now also R14.2, U$3.P$34; no longer R38.2, U$8.P$34
- net N$7: now also IC2.7, R47.2; no longer IC1.7, R16.2
- net N$8: now also C100.P$2, IC2.1, IC2.8, IC2.9; no longer C58.P$2, IC1.1, IC1.8, IC1.9
- net PGOOD: now also U$3.P$15; no longer U$8.P$15
- net PROM_TDO: now also U$10.P$17; no longer U$5.P$17
- net S1FB: now also C27.2, R27.1, R30.2, U$3.P$1; no longer C86.2, R26.1, R27.2, U$8.P$1
- net S1SW: now also L6.P$1, U$3.P$3, U$3.P$4; no longer L11.P$1, U$8.P$3, U$8.P$4
- net S3FB: now also C9.2, R16.1, R18.2, U$3.P$7; no longer C87.2, R28.1, R29.2, U$8.P$7
- net S3SW: now also L2.P$1, U$3.P$9; no longer L6.P$1, U$8.P$9
- net S4FB: now also C26.2, R26.1, R28.2, U$3.P$12; no longer C88.2, R30.1, R31.2, U$8.P$12
- net S4SW: now also L5.P$1, U$3.P$10; no longer L7.P$1, U$8.P$10
- net S5FB: now also C14.2, R19.1, R20.2, U$3.P$20; no longer C89.2, R32.1, R33.2, U$8.P$20
- net S5SW: now also L3.P$1, U$3.P$22, U$3.P$23; no longer L10.P$1, U$8.P$22, U$8.P$23
- net S7FB: now also C25.2, R25.1, R29.2, U$3.P$26; no longer C90.2, R34.1, R35.2, U$8.P$26
- net S7SW: now also L4.P$1, U$3.P$28; no longer L8.P$1, U$8.P$28
- net S8FB: now also C8.2, R15.1, R17.2, U$3.P$31; no longer C91.2, R36.1, R37.2, U$8.P$31
- net S8SW: now also L1.P$1, U$3.P$29; no longer L9.P$1, U$8.P$29
- net SIGNAL_IN: now also U$7.P$16, X3.1; no longer U$3.P$16, X1.1@1
- net S_TEMP: now also U$3.P$36; no longer U$8.P$36
- net VIN: now also C1.1, C12.1, C13.1, C15.1, C17.1, C2.1, C3.1, C4.1, C6.1, C7.1, U$3.P$11, U$3.P$17, U$3.P$2, U$3.P$21, U$3.P$24, U$3.P$25, U$3.P$27, U$3.P$30, U$3.P$33, U$3.P$35, U$3.P$5, U$3.P$6, U$3.P$8; no longer C70.1, C71.1, C72.1, C73.1, C74.1, C75.1, C76.1, C77.1, C78.1, C79.1, U$8.P$11, U$8.P$17, U$8.P$2, U$8.P$21, U$8.P$24, U$8.P$25, U$8.P$27, U$8.P$30, U$8.P$33, U$8.P$35, U$8.P$5, U$8.P$6, U$8.P$8

Commit message: Changed Ferrites plus some peripherals
Parts:
- removed C66, C67, C69, C70, C72, C73, C75: .1uF, Schuyler:0204REVERSE
- added C103, C104, C105, C106, C107, C108, C109, C110, C111, C112: .1uF, Schuyler:0204REVERSE
- added J2: MICRO-FIT_3.0_2POS_RA_SMD, Schuyler:MICRO-FIT_3.02POS_RA_SMD
- added L12: CHOKE_CM_ACM7060-301, Schuyler:ACM7060_CHOKE
- added L13: (no value), Schuyler:MURATA_BLM18
- added U$11: SLIDER_SPDT_1101M2S3AQE2, Schuyler:C_AND_K_1101M2S3AQE2
- C3: value 33uF -> 100uF; device SparkFun-Passives:0805 -> Schuyler:2917_MURATA_CAP
- C59, C64: value .1uF -> 10nF; device Schuyler:0204REVERSE -> rcl:C0201
- C63: value .1uF -> 1uF
- L10: device Schuyler:2220_FERRITE_BEAD -> Schuyler:MURATA_BLM18
- L7, L8, L9: value 400@100MHz -> (none); device Schuyler:2220_FERRITE_BEAD -> Schuyler:MURATA_BLM18
- moved C43 928.6 mm to (-179.6, -865.3), turned to 0 degrees
- moved C63 910.2 mm to (-223.1, -902.2)
- moved C46 878.5 mm to (-175.6, -865.3)
- moved C48 877.7 mm to (-177.6, -867.9)
- moved C53 876.9 mm to (-179.6, -870.5)
- moved C58 872.3 mm to (-175.6, -870.5)
- moved L7 851.5 mm to (-216.9, -899.0)
- moved L8 845.9 mm to (-219.1, -899.0)
- moved C64 830.8 mm to (-225.1, -905.4)
- moved C59 827.0 mm to (-221.3, -902.0)
- moved L10 821.1 mm to (-221.3, -899.0)
- moved L9 810.5 mm to (-225.2, -902.5)
- moved C54 787.1 mm to (-177.6, -870.5)
- moved C47 785.7 mm to (-179.6, -867.9)
- moved C49 784.5 mm to (-175.6, -867.9)
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Connections:
- new net N$1: L12.P$4, U$11.P$1
- new net N$17: C3.P$2, L13.P$1, U$11.P$2
- new net POWER_IN+: J2.P$2, L12.P$1
- new net POWER_IN-: J2.P$1, L12.P$2
- net 1V9A: now also C103.P$1, C104.P$1, C105.P$1, C106.P$1, C107.P$1, C108.P$1, C109.P$1, C110.P$1, C111.P$1, C112.P$1; no longer C43.P$1, C46.P$1, C48.P$1, C53.P$1, C58.P$1, C63.P$1, C66.P$1, C69.P$1, C72.P$1, C75.P$1
- net 1V9D: now also C43.P$1, C46.P$1, C48.P$1, C53.P$1, C58.P$1; no longer C59.P$1, C64.P$1, C67.P$1, C70.P$1, C73.P$1
- net 2V5A: now also C64.1
- net 3V3: now also C59.1, C63.P$1; no longer R42.2
- net AGND: now also C103.P$2, C104.P$2, C105.P$2, C106.P$2, C107.P$2, C108.P$2, C109.P$2, C110.P$2, C111.P$2, C112.P$2, C64.2; no longer C43.P$2, C46.P$2, C48.P$2, C53.P$2, C58.P$2, C63.P$2, C66.P$2, C69.P$2, C72.P$2, C75.P$2
- net DGND: now also C3.P$1, C43.P$2, C46.P$2, C48.P$2, C53.P$2, C58.P$2, C59.2, C63.P$2, L12.P$3, X1.G@1, X1.G@2, X1.G@3, X1.G@4; no longer C3.2, C59.P$2, C64.P$2, C67.P$2, C70.P$2, C73.P$2
- net FPGA_INITB: no longer R42.1
- net VIN: now also L13.P$2; no longer C3.1

Commit message: Unchecked Finalized Schematic
Parts:
- removed C16: NA, rcl:C0603
- added D1, D2, D3, D4, D5, D6: (no value), Schuyler:0603_LED
- added H1, H2, H3, H4: MOUNT-HOLE2.8, holes:2,8
- added JP2: M10", SparkFun-Connectors:1X10
- added JP3: (no value), SparkFun-Passives:1X02
- added R56, R57, R58, R59, R60: 330, rcl:R0201
- added R61: 50, rcl:R0201
- added R62: NA, rcl:R0603
- added TP10, TP11, TP12, TP13, TP14, TP15: TPPAD1-13, testpad:P1-13
- L11: value 600@100MHz -> (none); device dp_devices:FB603 -> Schuyler:MURATA_BLM18
- R23: value 806K -> 10k
- R24: value 150K -> 1k
- moved L11 667.3 mm to (-227.4, -910.6)
- moved R24 255.2 mm to (-229.9, -983.4)
- moved R23 188.1 mm to (-227.4, -918.4)
Connections:
- new net !RXLED: D2.CATHODE, IC2.11
- new net !TXLED: D3.CATHODE, IC2.5
- new net FPGA_GPIO0: JP2.1, U$2.P$46
- new net FPGA_GPIO1: JP2.2, U$2.P$57
- new net FPGA_GPIO2: JP2.3, U$2.P$58
- new net FPGA_GPIO3: JP2.4, U$2.P$59
- new net FPGA_GPIO4: JP2.5, U$2.P$61
- new net FPGA_GPIO5: D6.CATHODE, JP2.6, U$2.P$62
- new net FPGA_GPIO6: D5.CATHODE, JP2.7, U$2.P$64
- new net FPGA_GPIO7: D4.CATHODE, JP2.8, U$2.P$67
- new net N$10: D2.ANODE, R56.2
- new net N$19: D6.ANODE, R60.2
- new net N$21: D5.ANODE, R59.2
- new net N$22: D4.ANODE, R58.2
- new net N$26: U$2.P$108, U$2.P$91, U$2.P$96
- new net N$9: D1.ANODE, R24.1
- net 1V2: now also U$2.P$89
- net 1V8: now also U$2.P$77
- net 3V3: now also JP2.10, R58.1, R59.1, R60.1, U$2.P$90; no longer R23.2
- net 3V3S: now also TP14.TP
- net 5VUSB: now also L11.P$2; no longer L11.1
- net 5VUSB_CON: now also L11.P$1; no longer L11.2
- net DGND: now also D1.CATHODE, JP2.9, R61.1, R62.2; no longer C16.2, R24.2
- net FPGA_DONE: now also TP12.TP
- net FPGA_INITB: now also TP13.TP
- net GND: no longer U$2.P$108, U$2.P$77, U$2.P$91, U$2.P$96
- net N$1: now also JP3.2
- net N$13: now also D3.ANODE, R57.2; no longer C16.1, R23.1, R24.1, U$3.P$13
- net N$17: now also JP3.1, R24.2
- net N$8: now also R56.1, R57.1
- net PGOOD: now also R23.1, TP11.TP, U$2.P$45
- net S_TEMP: now also TP10.TP
- net TRIGGER: now also R61.2
- net TRIG_REF: now also R62.1, TP15.TP
- net VCCAUX: no longer U$2.P$90
- net VCCINT: no longer U$2.P$89
- net VIN: now also U$3.P$13
